File: mcxn_test_board/mcxn_test_board.kicad_sch (KiCad schematic)
At the start: 74 parts, among them J1 USB4085, J10 P4_GENERAL, J11 I2C, J12 MicroSD_socket, J13 KEYPAD, J14 5VDC IN, J2 SWD, J3 UART/CAN, J4 DISP/SPI, J5 P1MISC, J6 PDM_IN, J7 I2S_IN, J8 I2S_OUT, J9 P4/ADC, SW1 SKQGAFE010, SW2 SKQGAFE010, SW3 SKQGAFE010, SW4 BOOT, SW5 RESET, U1 MCXN236VKLT, U2 MIC5209-3.3YS, U3 SRV05-4, Y1 830108212309, Y2 830009678

Commit message: Add files via upload
Parts:
- added C28: 10u, User_Global_Library:Cap-Tant-CaseB, symbol Device:C_Polarized_Small
- added C29: 1u, Capacitor_SMD:C_0805_2012Metric, symbol Device:C_Small
- added R20: 0R, User_Global_Library:0402-footprint-improved-Res3D, symbol Device:R
- added TP10, TP11, TP8, TP9: 0V, User_Global_Library:TestPoint_Plated_Hole_0.6mm, symbol Connector:TestPoint_Small
- added U10, U11, U14, U8: (no value), User_Global_Library:bare-pad-2x1, symbol User_Global_Symbol_Library:PAD
- added U13, U16, U17, U4, U5, U9: (no value), User_Global_Library:bare-pad-3x3, symbol User_Global_Symbol_Library:PAD
- added U6, U7: (no value), User_Global_Library:bare-pad-2x2, symbol User_Global_Symbol_Library:PAD
- C16: value 1u -> 100n; footprint User_Global_Library:0603-footprint-improved-Cap3D -> User_Global_Library:0402-footprint-improved-Cap3D
Connections:
- net 0V: now also C28.2, C29.2, TP10.1, TP11.1, TP8.1, TP9.1
- net at C10.1, FB1.2, U1.31 (VREFH): now also C28.1, C29.1, R20.2; no longer C16.1, U1.30 (VDD_ANA)
- new net: C16.1, R20.1, U1.30 (VDD_ANA)
Other:
- note added: "BARE PADS"
- moved on the sheet: C10, C18, C21, C22, D3, D4, FB1, J14, U2

Commit message: Add files via upload
Other:
- note added: "0.1"
- note removed: "1"
Changed lines of the file:
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@@
 		)
 	)
-	(text "1"
+	(text "0.1"
 		(exclude_from_sim no)
-		(at 394.208 278.638 0)
+		(at 396.24 278.638 0)
 		(effects
 			(font
