File: mcxn_test_board/mcxn_test_board.kicad_pcb (KiCad board)
At the start: 4 copper layers, 70 x 70 mm, 74 parts, among them J1 USB4085, J10 P4_GENERAL, J11 I2C, J12 MicroSD_socket, J13 KEYPAD, J14 5VDC IN, J2 SWD, J3 UART/CAN, J4 DISP/SPI, J5 P1MISC, J6 PDM_IN, J7 I2S_IN, J8 I2S_OUT, J9 P4/ADC, SW1 SKQGAFE010, SW2 SKQGAFE010, SW3 SKQGAFE010, SW4 BOOT, SW5 RESET, U1 MCXN236VKLT, U2 MIC5209-3.3YS, U3 SRV05-4, Y1 830108212309, Y2 830009678

Commit message: Add files via upload
Parts:
- added C28: 10u, User_Global_Library:Cap-Tant-CaseB, F.Cu at (92.0, 74.8)
- added C29: 1u, Capacitor_SMD:C_0805_2012Metric, F.Cu at (93.0, 72.0)
- added R20: 0R, User_Global_Library:0402-footprint-improved-Res3D, F.Cu at (95.8, 71.0)
- added TP10: 0V, User_Global_Library:TestPoint_Plated_Hole_0.6mm, F.Cu at (77.3, 84.4)
- added TP11: 0V, User_Global_Library:TestPoint_Plated_Hole_0.6mm, F.Cu at (76.4, 47.3)
- added TP8: 0V, User_Global_Library:TestPoint_Plated_Hole_0.6mm, F.Cu at (89.5, 72.1)
- added TP9: 0V, User_Global_Library:TestPoint_Plated_Hole_0.6mm, F.Cu at (89.1, 81.0)
- added U10: ~, User_Global_Library:bare-pad-2x1, F.Cu at (86.0, 67.6)
- added U11: ~, User_Global_Library:bare-pad-2x1, F.Cu at (86.7, 83.5)
- added U13: ~, User_Global_Library:bare-pad-3x3, F.Cu at (79.7, 67.6)
- added U14: ~, User_Global_Library:bare-pad-2x1, F.Cu at (83.5, 70.2)
- added U16: ~, User_Global_Library:bare-pad-3x3, F.Cu at (83.5, 67.6)
- added U17: ~, User_Global_Library:bare-pad-3x3, F.Cu at (79.7, 71.4)
- added U4: ~, User_Global_Library:bare-pad-3x3, F.Cu at (84.1, 83.5)
- added U5: ~, User_Global_Library:bare-pad-3x3, F.Cu at (85.4, 79.7)
- added U6: ~, User_Global_Library:bare-pad-2x2, F.Cu at (82.9, 81.0)
- added U7: ~, User_Global_Library:bare-pad-2x2, F.Cu at (86.7, 77.1)
- added U8: ~, User_Global_Library:bare-pad-2x1, F.Cu at (87.9, 78.4)
- added U9: ~, User_Global_Library:bare-pad-3x3, F.Cu at (80.3, 83.5)
- C16: value 1u -> 100n; footprint User_Global_Library:0603-footprint-improved-Cap3D -> User_Global_Library:0402-footprint-improved-Cap3D
- moved FB1 3.05 mm to (91.8, 78.2), turned to 45 degrees
- moved C15 2.83 mm to (97.2, 72.9)
- moved C16 2.19 mm to (93.9, 70.3), turned to 180 degrees
- moved C10 0.75 mm to (96.6, 70.0), turned to 0 degrees
- moved C7 0.62 mm to (98.4, 70.2)
Connections:
- C10 pad 1: Net-(U1PWR-VDD_ANA) -> Net-(U1PWR-VREFH)
- FB1 pad 2: Net-(U1PWR-VDD_ANA) -> Net-(U1PWR-VREFH)
- U1 pad 31: Net-(U1PWR-VDD_ANA) -> Net-(U1PWR-VREFH)
Routing:
- net Net-(U1PWR-VDD_ANA): track 13.5 -> 4.68 mm
- net +3.3V: track 91.3 -> 82.9 mm, vias 19 -> 21
- net Net-(U1PWR-VREFH): track 0.00 -> 3.99 mm
- net 0V: track 88.4 -> 89.6 mm, vias 46 -> 52
- net /P4_4: track 34.2 -> 33.6 mm
- net /P4_3: track 30.0 -> 29.4 mm
- net /P4_12: track 33.1 -> 33.7 mm
- added copper zone on F.Cu, net Net-(U1PWR-VREFH)
Other:
- outline, holes or cut-outs redrawn
- board text added: "EZ-MXCN"
- board text added: "MCXN236/235/547 VKLT TEST BOARD"
- board text removed: "MCXN235/236/ 547VKLT TEST BOARD"

Commit message: Add files via upload
Other:
- board text added: "EZ-MCXN"
- board text removed: "EZ-MXCN"
Changed lines of the file:
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@@
 		)
 	)
-	(gr_text "EZ-MXCN"
+	(gr_text "EZ-MCXN"
 		(at 83.744 44.125 90)
 		(layer "F.SilkS")
@@
 	)
 	(segment
+		(start 96.1809 70)
+		(end 96.1809 69.6191)
+		(width 0.2032)
+		(layer "F.Cu")
+		(net "Net-(U1PWR-VREFH)")
+	)
+	(segment
+		(start 96.1809 69.6191)
+		(end 96.5 69.3)
+		(width 0.2032)
+		(layer "F.Cu")
+		(net "Net-(U1PWR-VREFH)")
+	)
+	(segment
+		(start 96.5 69.3)
+		(end 96.5 67.75)
+		(width 0.2032)
+		(layer "F.Cu")
+		(net "Net-(U1PWR-VREFH)")
+	)
+	(segment
+		(start 96.2 71)
+		(end 96.2 71.6)
+		(width 0.27)
+		(layer "F.Cu")
+		(net "Net-(U1PWR-VREFH)")
+	)
+	(segment
+		(start 96.2 70.0191)
+		(end 96.1809 70)
+		(width 0.2032)
+		(layer "F.Cu")
+		(net "Net-(U1PWR-VREFH)")
+	)
+	(segment
+		(start 96.2 71)
+		(end 96.2 70.0191)
+		(width 0.2032)
+		(layer "F.Cu")
+		(net "Net-(U1PWR-VREFH)")
+	)
+	(segment
 		(start 117.405841 45.75)
 		(end 119.939 45.75)
@@
 	)
 	(segment
-		(start 94.71542 70.3)
-		(end 95.10771 69.90771)
-		(width 0.2032)
-		(layer "F.Cu")
-		(net "Net-(U1PWR-VDD_ANA)")
-	)
-	(segment
-		(start 95.3618 71)
-		(end 95.3618 70.1618)
-		(width 0.2032)
-		(layer "F.Cu")
-		(net "Net-(U1PWR-VDD_ANA)")
-	)
-	(segment
-		(start 94.3191 70.3)
-		(end 94.71542 70.3)
-		(width 0.2032)
-		(layer "F.Cu")
-		(net "Net-(U1PWR-VDD_ANA)")
-	)
-	(segment
-		(start 96 69.01542)
-		(end 96 67.75)
-		(width 0.2032)
-		(layer "F.Cu")
-		(net "Net-(U1PWR-VDD_ANA)")
-	)
-	(segment
-		(start 95.10771 69.90771)
-		(end 95.3618 69.65362)
-		(width 0.2032)
-		(layer "F.Cu")
-		(net "Net-(U1PWR-VDD_ANA)")
-	)
-	(segment
-		(start 95.3618 69.65362)
-		(end 96 69.01542)
-		(width 0.2032)
-		(layer "F.Cu")
-		(net "Net-(U1PWR-VDD_ANA)")
-	)
-	(segment
-		(start 95.3618 70.1618)
-		(end 95.10771 69.90771)
-		(width 0.2032)
-		(layer "F.Cu")
-		(net "Net-(U1PWR-VDD_ANA)")
-	)
-	(segment
 		(start 85.52898 86.4436)
 		(end 97.48629 74.48629)
@@
 	)
 	(segment
+		(start 94.71542 70.3)
+		(end 95.10771 69.90771)
+		(width 0.2032)
+		(layer "F.Cu")
+		(net "Net-(U1PWR-VDD_ANA)")
+	)
+	(segment
+		(start 95.3618 71)
+		(end 95.3618 70.1618)
+		(width 0.2032)
+		(layer "F.Cu")
+		(net "Net-(U1PWR-VDD_ANA)")
+	)
+	(segment
+		(start 94.3191 70.3)
+		(end 94.71542 70.3)
+		(width 0.2032)
+		(layer "F.Cu")
+		(net "Net-(U1PWR-VDD_ANA)")
+	)
+	(segment
+		(start 96 69.01542)
+		(end 96 67.75)
+		(width 0.2032)
+		(layer "F.Cu")
+		(net "Net-(U1PWR-VDD_ANA)")
+	)
+	(segment
+		(start 95.10771 69.90771)
+		(end 95.3618 69.65362)
+		(width 0.2032)
+		(layer "F.Cu")
+		(net "Net-(U1PWR-VDD_ANA)")
+	)
+	(segment
+		(start 95.3618 69.65362)
+		(end 96 69.01542)
+		(width 0.2032)
+		(layer "F.Cu")
+		(net "Net-(U1PWR-VDD_ANA)")
+	)
+	(segment
+		(start 95.3618 70.1618)
+		(end 95.10771 69.90771)
+		(width 0.2032)
+		(layer "F.Cu")
+		(net "Net-(U1PWR-VDD_ANA)")
+	)
+	(segment
 		(start 107.75 66)
 		(end 107.75 66.75)
@@
 		(net "/P1_2")
 	)
-	(segment
-		(start 96.1809 70)
-		(end 96.1809 69.6191)
-		(width 0.2032)
-		(layer "F.Cu")
-		(net "Net-(U1PWR-VREFH)")
-	)
-	(segment
-		(start 96.1809 69.6191)
-		(end 96.5 69.3)
-		(width 0.2032)
-		(layer "F.Cu")
-		(net "Net-(U1PWR-VREFH)")
-	)
-	(segment
-		(start 96.5 69.3)
-		(end 96.5 67.75)
-		(width 0.2032)
-		(layer "F.Cu")
-		(net "Net-(U1PWR-VREFH)")
-	)
-	(segment
-		(start 96.2 71)
-		(end 96.2 71.6)
-		(width 0.27)
-		(layer "F.Cu")
-		(net "Net-(U1PWR-VREFH)")
-	)
-	(segment
-		(start 96.2 70.0191)
-		(end 96.1809 70)
-		(width 0.2032)
-		(layer "F.Cu")
-		(net "Net-(U1PWR-VREFH)")
-	)
-	(segment
-		(start 96.2 71)
-		(end 96.2 70.0191)
-		(width 0.2032)
-		(layer "F.Cu")
-		(net "Net-(U1PWR-VREFH)")
-	)
 	(zone

Commit message: Add files via upload
Routing:
- net 0V: track 89.6 -> 131.9 mm
- net /COL1: track 55.5 -> 50.5 mm
- net Net-(U1PWR-VDD_CORE_1): track 48.9 -> 49.5 mm
