File: mcxn_mini_board/mcxn_mini_board.kicad_sch (KiCad schematic)
At the start: 46 parts, among them J1 USB4085, J2 SWD, J3 MIC_A, J4 MIC_B, J5 FFC_0.5MM, SW1 SKQGAFE010, SW2 SKQGAFE010, SW3 SKQGAFE010, SW4 BOOT, SW5 RESET, U1 MCXN236VKLT, U2 MIC5209-3.3YS, U3 SRV05-4, Y1 830108212309

Commit message: Add files via upload
Connections:
- net 0V: now also J2.3 (Pin_3); no longer J2.1 (Pin_1)
- net SWC: now also J2.2 (Pin_2); no longer J2.3 (Pin_3)
- net SWD: now also J2.1 (Pin_1); no longer J2.2 (Pin_2)
Changed lines of the file:
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@@
 	)
 	(bus_entry
-		(at 160.02 184.15)
+		(at 160.02 186.69)
 		(size -2.54 -2.54)
 		(stroke
@@
 	)
 	(bus_entry
-		(at 160.02 186.69)
+		(at 160.02 189.23)
 		(size -2.54 -2.54)
 		(stroke
@@
 		)
 	)
-	(bus
-		(pts
-			(xy 160.02 181.61) (xy 160.02 193.04)
-		)
-		(stroke
-			(width 0)
-			(type default)
-		)
-	)
 	(wire
 		(pts
@@
 	(wire
 		(pts
-			(xy 152.4 184.15) (xy 157.48 184.15)
+			(xy 152.4 186.69) (xy 157.48 186.69)
 		)
 		(stroke
@@
 	(wire
 		(pts
-			(xy 153.67 186.69) (xy 153.67 187.96)
-		)
-		(stroke
-			(width 0)
-			(type default)
-		)
-	)
-	(wire
-		(pts
 			(xy 151.13 156.21) (xy 151.13 161.29)
 		)
@@
 	(wire
 		(pts
+			(xy 162.56 181.61) (xy 162.56 182.88)
+		)
+		(stroke
+			(width 0)
+			(type default)
+		)
+	)
+	(wire
+		(pts
 			(xy 120.65 171.45) (xy 124.46 171.45)
 		)
@@
 	(wire
 		(pts
+			(xy 152.4 181.61) (xy 162.56 181.61)
+		)
+		(stroke
+			(width 0)
+			(type default)
+		)
+	)
+	(wire
+		(pts
 			(xy 60.96 80.01) (xy 64.77 80.01)
 		)
@@
 	(wire
 		(pts
-			(xy 152.4 186.69) (xy 153.67 186.69)
-		)
-		(stroke
-			(width 0)
-			(type default)
-		)
-	)
-	(wire
-		(pts
 			(xy 41.91 33.02) (xy 53.34 33.02)
 		)
@@
 	(wire
 		(pts
-			(xy 152.4 181.61) (xy 157.48 181.61)
+			(xy 152.4 184.15) (xy 157.48 184.15)
 		)
 		(stroke
@@
 		)
 	)
+	(bus
+		(pts
+			(xy 160.02 185.42) (xy 160.02 193.04)
+		)
+		(stroke
+			(width 0)
+			(type default)
+		)
+	)
 	(wire
 		(pts
@@
 	)
 	(label "SWC"
-		(at 152.4 181.61 0)
+		(at 152.4 184.15 0)
 		(effects
 			(font
@@
 	)
 	(label "SWD"
-		(at 152.4 184.15 0)
+		(at 152.4 186.69 0)
 		(effects
 			(font
@@
 	(symbol
 		(lib_id "User_Global_Symbol_Library:0V")
-		(at 153.67 187.96 0)
+		(at 162.56 182.88 0)
 		(unit 1)
 		(body_style 1)
@@
 		(dnp no)
 		(property "Reference" "#PWR040"
-			(at 153.67 193.04 0)
+			(at 162.56 187.96 0)
 			(hide yes)
 			(show_name no)
@@
 		)
 		(property "Value" "0V"
-			(at 153.67 190.754 0)
+			(at 162.56 185.674 0)
 			(show_name no)
 			(do_not_autoplace no)
@@
 		)
 		(property "Footprint" ""
-			(at 153.67 187.96 0)
+			(at 162.56 182.88 0)
 			(hide yes)
 			(show_name no)
@@
 		)
 		(property "Datasheet" ""
-			(at 153.67 187.96 0)
+			(at 162.56 182.88 0)
 			(hide yes)
 			(show_name no)
@@
 		)
 		(property "Description" "Power symbol creates a global label with name \"0V\""
-			(at 153.67 187.96 0)
+			(at 162.56 182.88 0)
 			(hide yes)
 			(show_name no)
