File: mcxn_mini_board/mcxn_mini_board.kicad_pcb (KiCad board)
At the start: 4 copper layers, 26 x 48 mm, 46 parts, among them J1 USB4085, J2 SWD, J3 MIC_A, J4 MIC_B, J5 FFC_0.5MM, SW1 SKQGAFE010, SW2 SKQGAFE010, SW3 SKQGAFE010, SW4 BOOT, SW5 RESET, U1 MCXN236VKLT, U2 MIC5209-3.3YS, U3 SRV05-4, Y1 830108212309

Commit message: Add files via upload
Connections:
- J2 pad 1: 0V -> /SWD
- J2 pad 2: /SWD -> /SWC
- J2 pad 3: /SWC -> 0V
Routing:
- net 0V: track 123.7 -> 126.1 mm
- net /SWC: track 26.0 -> 27.1 mm
- net /SWD: track 26.9 -> 27.9 mm
Other:
- board text added: "0"
- board text added: "3"
- board text added: "D"
- board text added: "MIC-A"
- board text added: "MIC-B"
- board text added: "VB"

Commit message: Add files via upload
Routing:
- net 0V: vias 59 -> 63
Changed lines of the file:
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@@
 		(sheetname "/")
 		(sheetfile "mcxn_mini_board.kicad_sch")
-		(units
-			(unit
-				(name "PWR")
-				(pins "13" "96" "83" "73" "66" "59" "34" "55" "30" "31" "32" "47" "44"
-					"12" "58" "53" "54" "33" "52" "50" "43" "EP"
-				)
-			)
-			(unit
-				(name "USB/DEBUG")
-				(pins "82" "42" "41" "40" "10" "11" "4" "3" "2" "1" "46" "45" "49" "48"
-					"9" "78" "77" "76"
-				)
-			)
-			(unit
-				(name "UI")
-				(pins "70" "69" "68" "67" "65" "64" "63" "62" "61" "75" "94" "93" "92"
-					"57" "60" "56" "72" "74"
-				)
-			)
-			(unit
-				(name "AUDIO")
-				(pins "80" "81" "86" "14" "15" "17" "18" "20" "21" "16" "19" "71")
-			)
-			(unit
-				(name "UNUSED")
-				(pins "5" "6" "7" "8" "22" "23" "24" "25" "26" "27" "28" "29" "35" "36"
-					"37" "38" "39" "100" "99" "98" "97" "95" "87" "79" "51"
-				)
-			)
-			(unit
-				(name "SPI/I2C")
-				(pins "91" "88" "89" "90" "85" "84")
-			)
-		)
 		(attr smd)
 		(duplicate_pad_numbers_are_jumpers no)
@@
 		(pad "EP" thru_hole circle
 			(at -2.2225 -0.9525)
-			(size 0.9 0.9)
-			(drill 0.3)
+			(size 1 1)
+			(drill 0.4)
 			(layers "*.Cu" "*.Mask")
 			(remove_unused_layers no)
@@
 		(pad "EP" thru_hole circle
 			(at -2.2225 0.9525)
-			(size 0.9 0.9)
-			(drill 0.3)
+			(size 1 1)
+			(drill 0.4)
 			(layers "*.Cu" "*.Mask")
 			(remove_unused_layers no)
@@
 		(pad "EP" thru_hole circle
 			(at -0.9525 -2.2225)
-			(size 0.9 0.9)
-			(drill 0.3)
+			(size 1 1)
+			(drill 0.4)
 			(layers "*.Cu" "*.Mask")
 			(remove_unused_layers no)
@@
 		(pad "EP" thru_hole circle
 			(at -0.9525 2.2225)
-			(size 0.9 0.9)
-			(drill 0.3)
+			(size 1 1)
+			(drill 0.4)
 			(layers "*.Cu" "*.Mask")
 			(remove_unused_layers no)
@@
 		(pad "EP" thru_hole circle
 			(at -0.95 -0.95)
-			(size 0.9 0.9)
-			(drill 0.3)
+			(size 1 1)
+			(drill 0.4)
 			(layers "*.Cu" "*.Mask")
 			(remove_unused_layers no)
@@
 		(pad "EP" thru_hole circle
 			(at -0.95 0.95)
-			(size 0.9 0.9)
-			(drill 0.3)
+			(size 1 1)
+			(drill 0.4)
 			(layers "*.Cu" "*.Mask")
 			(remove_unused_layers no)
@@
 		(pad "EP" thru_hole circle
 			(at 0.95 -0.95)
-			(size 0.9 0.9)
-			(drill 0.3)
+			(size 1 1)
+			(drill 0.4)
 			(layers "*.Cu" "*.Mask")
 			(remove_unused_layers no)
@@
 		(pad "EP" thru_hole circle
 			(at 0.95 0.95)
-			(size 0.9 0.9)
-			(drill 0.3)
+			(size 1 1)
+			(drill 0.4)
 			(layers "*.Cu" "*.Mask")
 			(remove_unused_layers no)
@@
 		(pad "EP" thru_hole circle
 			(at 0.9525 -2.2225)
-			(size 0.9 0.9)
-			(drill 0.3)
+			(size 1 1)
+			(drill 0.4)
 			(layers "*.Cu" "*.Mask")
 			(remove_unused_layers no)
@@
 		(pad "EP" thru_hole circle
 			(at 0.9525 2.2225)
-			(size 0.9 0.9)
-			(drill 0.3)
+			(size 1 1)
+			(drill 0.4)
 			(layers "*.Cu" "*.Mask")
 			(remove_unused_layers no)
@@
 		(pad "EP" thru_hole circle
 			(at 2.2225 -0.9525)
-			(size 0.9 0.9)
-			(drill 0.3)
+			(size 1 1)
+			(drill 0.4)
 			(layers "*.Cu" "*.Mask")
 			(remove_unused_layers no)
@@
 		(pad "EP" thru_hole circle
 			(at 2.2225 0.9525)
-			(size 0.9 0.9)
-			(drill 0.3)
+			(size 1 1)
+			(drill 0.4)
 			(layers "*.Cu" "*.Mask")
 			(remove_unused_layers no)
@@
 	)
 	(via
+		(at 93.3 62.4)
+		(size 0.7048)
+		(drill 0.4)
+		(layers "F.Cu" "B.Cu")
+		(free yes)
+		(net "0V")
+	)
+	(via
 		(at 108.75 59.5)
 		(size 0.7048)
@@
 	)
 	(via
+		(at 95.2 57.2)
+		(size 0.7048)
+		(drill 0.4)
+		(layers "F.Cu" "B.Cu")
+		(free yes)
+		(net "0V")
+	)
+	(via
+		(at 97.9 64.8)
+		(size 0.7048)
+		(drill 0.4)
+		(layers "F.Cu" "B.Cu")
+		(free yes)
+		(net "0V")
+	)
+	(via
 		(at 88.3094 66)
 		(size 0.7048)
@@
 		(net "0V")
 	)
+	(via
+		(at 103.9 58)
+		(size 0.7048)
+		(drill 0.4)
+		(layers "F.Cu" "B.Cu")
+		(free yes)
+		(net "0V")
+	)
